Commit message: added localizer

File: src/my_bot/description/camera.xacro (robot description, xacro)
@@ -1,5 +1,5 @@
 <?xml version="1.0"?>
 <robot xmlns:xacro="http://www.ros.org/wiki/xacro">
-    <joint name="camera_joint" type= "fixed">
+    <joint name="camera_joint" type="fixed">
         <parent link="chassis"/>
         <child link="camera_link"/>
@@ -15,5 +15,5 @@
     </link>
     <!--Extra linking for orientation compensation-->
-    <joint name="camera_optical_joint" type= "fixed">
+    <joint name="camera_optical_joint" type="fixed">
         <parent link="camera_link"/>
         <child link="camera_link_optical"/>
@@ -23,14 +23,14 @@
     <gazebo reference="camera_link">
         <material>Gazebo/Green</material>
-        <sensor name="camera" type="camera">
-            <pose> 0 0 0 0 0 0 </pose>
+        <sensor name="camera" type="depth">
+            <pose>0 0 0 0 0 0</pose>
             <visualize>true</visualize>
-            <update_rate>100</update_rate>
+            <update_rate>10</update_rate>
             <camera>
                 <horizontal_fov>1.089</horizontal_fov>
                 <image>
                     <format>R8G8B8</format>
-                    <width>1920</width>
-                    <height>1080</height>
+                    <width>640</width>
+                    <height>480</height>
                 </image>
                 <clip>
@@ -41,4 +41,6 @@
             <plugin name="camera_controller" filename="libgazebo_ros_camera.so">
                 <frame_name>camera_link_optical</frame_name>
+                <min_depth>0.1</min_depth>
+                <max_depth>8.0</max_depth>
             </plugin>
         </sensor>
